File: 2Phase_SynchBuck.kicad_sch (KiCad schematic)
At the start: 0 parts

Commit message: Update sch v1.0
Other:
- note added: "Digitally Controlled Power Conversion with STM32G474"
- note removed: "Digital Power Conversion with STM32G4"
