File: Interface_interconnects.kicad_sch (KiCad schematic)
At the start: 52 parts, among them CN701 USB4215-03-A, CN702 Conn_JTAG_STDC10, CN703 FFC2B28-16-G, CN704 FFC2B28-04-G, U701 USBLC6-2SC6

Commit message: Modified part number
Added 2nd Supplier
Added 2nd Mfr, Mfr NO.
Parts:
- R702, R703: Manufacturer 2nd (none) -> ROYALOHM; Manufacturer Part Number 2nd (none) -> 0402WGF5111TCE; Supplier 2nd (none) -> Electronisc Source; Supplier Part Number 2nd (none) -> 0150-3609-4
