File: Interface_interconnects.kicad_sch (KiCad schematic)
At the start: 52 parts, among them CN701 USB4215-03-A, CN702 Conn_JTAG_STDC10, CN703 FFC2B28-16-G, CN704 FFC2B28-04-G, U701 USBLC6-2SC6

Commit message: Updated Schematic v1.0
Parts:
- C705, C706: now left out of the parts list
Changed lines of the file:
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@@
 			(width 0)
 			(type default)
+			(color 255 0 0 1)
 		)
 	)
@@
 			(width 0)
 			(type default)
+			(color 255 0 0 1)
 		)
 	)
@@
 		(body_style 1)
 		(exclude_from_sim no)
-		(in_bom yes)
+		(in_bom no)
 		(on_board yes)
 		(in_pos_files yes)
@@
 		(body_style 1)
 		(exclude_from_sim no)
-		(in_bom yes)
+		(in_bom no)
 		(on_board yes)
 		(in_pos_files yes)
