File: Interface_interconnects.kicad_sch (KiCad schematic)
At the start: 52 parts, among them CN701 USB4215-03-A, CN702 Conn_JTAG_STDC10, CN703 FFC2B28-16-G, CN704 FFC2B28-04-G, U701 USBLC6-2SC6

Commit message: Migrate Symbol Librarys
Parts:
- CN701: symbol 0_connectors:USB_C_Receptacle_USB2.0_16P -> 0_Connectors:USB_C_Receptacle_USB2.0_16P
- CN702: symbol 0_connectors:Conn_JTAG_STDC10 -> 0_Connectors:Conn_JTAG_STDC10
- CN703: symbol 0_connectors:Conn_01x16_MountingPin -> 0_Connectors:Conn_01x16_MountingPin
- CN704: symbol 0_connectors:Conn_01x04_MountingPin -> 0_Connectors:Conn_01x04_MountingPin
- D701, D705, D706: symbol 0_protection:SP3031-01ETG -> 0_Protection:SP3031-01ETG
- D702, D703, D704: symbol 0_protection:PUSB3FR4Z -> 0_Protection:PUSB3FR4Z
- U701: symbol 0_protection:USBLC6-2SC6 -> 0_Protection:USBLC6-2SC6
Connections:
- no-connect marks 6 -> 5
Changed lines of the file:
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@@
 	)
 	(no_connect
-		(at 110.49 205.74)
-	)
-	(no_connect
 		(at 99.06 76.2)
 	)
@@
 	)
 	(symbol
-		(lib_id "0_connectors:Conn_01x04_MountingPin")
+		(lib_id "0_Connectors:Conn_01x04_MountingPin")
 		(at 229.87 176.53 0)
 		(mirror y)
@@
 	)
 	(symbol
-		(lib_id "0_protection:SP3031-01ETG")
+		(lib_id "0_Protection:SP3031-01ETG")
 		(at 113.03 165.1 270)
 		(unit 1)
@@
 	)
 	(symbol
-		(lib_id "0_protection:PUSB3FR4Z")
+		(lib_id "0_Protection:PUSB3FR4Z")
 		(at 110.49 210.82 0)
 		(unit 1)
@@
 	)
 	(symbol
-		(lib_id "0_protection:SP3031-01ETG")
+		(lib_id "0_Protection:SP3031-01ETG")
 		(at 251.46 186.69 270)
 		(unit 1)
@@
 	)
 	(symbol
-		(lib_id "0_protection:SP3031-01ETG")
+		(lib_id "0_Protection:SP3031-01ETG")
 		(at 251.46 158.75 270)
 		(unit 1)
@@
 	)
 	(symbol
-		(lib_id "0_protection:USBLC6-2SC6")
+		(lib_id "0_Protection:USBLC6-2SC6")
 		(at 116.84 83.82 0)
 		(unit 1)
@@
 	)
 	(symbol
-		(lib_id "0_protection:PUSB3FR4Z")
+		(lib_id "0_Protection:PUSB3FR4Z")
 		(at 295.91 104.14 0)
 		(unit 1)
@@
 	)
 	(symbol
-		(lib_id "0_connectors:Conn_JTAG_STDC10")
+		(lib_id "0_Connectors:Conn_JTAG_STDC10")
 		(at 86.36 190.5 0)
 		(unit 1)
@@
 	)
 	(symbol
-		(lib_id "0_connectors:Conn_01x16_MountingPin")
+		(lib_id "0_Connectors:Conn_01x16_MountingPin")
 		(at 240.03 77.47 0)
 		(mirror y)
@@
 	)
 	(symbol
-		(lib_id "0_protection:PUSB3FR4Z")
+		(lib_id "0_Protection:PUSB3FR4Z")
 		(at 273.05 104.14 0)
 		(unit 1)
@@
 	)
 	(symbol
-		(lib_id "0_connectors:USB_C_Receptacle_USB2.0_16P")
+		(lib_id "0_Connectors:USB_C_Receptacle_USB2.0_16P")
 		(at 83.82 83.82 0)
 		(unit 1)
