File: MCU_IOs.kicad_sch (KiCad schematic)
At the start: 13 parts, among them U401 STM32G474RET6, X501 ABM11W-24MHz-8

Commit message: Modified part number
Added 2nd Supplier
Added 2nd Mfr, Mfr NO.
Parts:
- C501, C502: Manufacturer 2nd (none) -> Murata; Manufacturer Part Number 2nd (none) -> GRM1555C1H6R8BA01D; Supplier 2nd (none) -> Electronisc Source; Supplier Part Number 2nd (none) -> 0160-0503-6
- R502: Manufacturer 2nd (none) -> ROYALOHM; Manufacturer Part Number 2nd (none) -> 0402WGF1001TCE; Supplier 2nd (none) -> Electronisc Source; Supplier Part Number 2nd (none) -> 0150-3602-3
- R507, R508: Manufacturer 2nd (none) -> ROYALOHM; Manufacturer Part Number 2nd (none) -> 0402WGF499JTCE; Supplier 2nd (none) -> Electronisc Source; Supplier Part Number 2nd (none) -> 0150-4765-9
