File: MCU_IOs.kicad_sch (KiCad schematic)
At the start: 13 parts, among them U401 STM32G474RET6, X501 ABM11W-24MHz-8

Commit message: Migrate Symbol Librarys
Parts:
- X501: symbol 0_crystal:Crystal_GND24 -> 0_Crystal:Crystal_GND24
Changed lines of the file:
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@@
 	)
 	(symbol
-		(lib_id "0_crystal:Crystal_GND24")
+		(lib_id "0_Crystal:Crystal_GND24")
 		(at 177.8 175.26 0)
 		(unit 1)
