File: analog_frontEnd.kicad_sch (KiCad schematic)
At the start: 18 parts, among them U601 TLV9061SIDBVR, U602 TLV9061SIDBVR

Commit message: Modified part number
Added 2nd Supplier
Added 2nd Mfr, Mfr NO.
Parts:
- C601, C602, C603, C605: Manufacturer 2nd (none) -> KYOCERA AVX; Manufacturer Part Number 2nd (none) -> 04025A470JAT2A; Supplier 2nd (none) -> Electronisc Source; Supplier Part Number 2nd (none) -> 0092-0407-5
- C604: Manufacturer 2nd (none) -> Murata; Manufacturer Part Number 2nd (none) -> GRM1555C1H102JA01D; Supplier 2nd (none) -> Electronisc Source; Supplier Part Number 2nd (none) -> 0160-0208-1
- R601, R602, R603, R605: Manufacturer 2nd (none) -> ROYALOHM; Manufacturer Part Number 2nd (none) -> 0402WGF499JTCE; Supplier 2nd (none) -> Electronisc Source; Supplier Part Number 2nd (none) -> 0150-4765-9
- R604: Manufacturer 2nd (none) -> ROYALOHM; Manufacturer Part Number 2nd (none) -> CQ02WGF1000TCE; Supplier 2nd (none) -> Electronisc Source; Supplier Part Number 2nd (none) -> 0150-4399-1
