File: analog_frontEnd.kicad_sch (KiCad schematic)
At the start: 18 parts, among them U601 TLV9061SIDBVR, U602 TLV9061SIDBVR

Commit message: Update revision
- Shc.
- Render images
Parts:
- U601, U602: value TLV9061SIDBVR -> TLV9061IDBVR; Manufacturer Part Number TLV9061SIDBVR -> TLV9061IDBVR; Supplier Part Number 296-53200-1-ND -> 296-52284-1-ND
Other:
- note removed: "No buffer and short this JP: t_{settling} = ~4us"
- note removed: "t_{ACQ} must greater than t_{settling} for accuracy."
Changed lines of the file:
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@@
 		)
 	)
-	(text "No buffer and short this JP: t_{settling} = ~4us"
-		(exclude_from_sim no)
-		(at 285.75 226.06 0)
-		(effects
-			(font
-				(size 1.5 1.5)
-			)
-		)
-	)
-	(text "t_{ACQ} must greater than t_{settling} for accuracy."
-		(exclude_from_sim no)
-		(at 276.86 134.62 0)
-		(effects
-			(font
-				(size 1.778 1.778)
-				(thickness 0.3556)
-				(bold yes)
-				(italic yes)
-				(color 194 0 0 1)
-			)
-		)
-	)
 	(text "t_{settling} = ~450ns"
 		(exclude_from_sim no)
@@
 	(text_box "LAYOUT NOTE:\n\nPlacing OpAmp and RC Filter close to the ADC input or Analog Zone"
 		(exclude_from_sim no)
-		(at 235.2492 117.7806 0)
+		(at 235.2492 125.4006 0)
 		(size 40.3408 10.4894)
 		(margins 0.9525 0.9525 0.9525 0.9525)
@@
 	(text_box "LAYOUT NOTE:\n\nRount away from magnetic compenents"
 		(exclude_from_sim no)
-		(at 278.13 118.11 0)
+		(at 278.13 125.73 0)
 		(size 40.3408 10.0062)
 		(margins 0.9525 0.9525 0.9525 0.9525)
@@
 			)
 		)
-		(property "Value" "TLV9061SIDBVR"
+		(property "Value" "TLV9061IDBVR"
 			(at 295.91 85.09 0)
 			(show_name no)
@@
 			)
 		)
-		(property "Manufacturer Part Number" "TLV9061SIDBVR"
+		(property "Manufacturer Part Number" "TLV9061IDBVR"
 			(at 289.56 90.17 0)
 			(hide yes)
@@
 			)
 		)
-		(property "Supplier Part Number" "296-53200-1-ND"
+		(property "Supplier Part Number" "296-52284-1-ND"
 			(at 289.56 90.17 0)
 			(hide yes)
@@
 			)
 		)
-		(property "Value" "TLV9061SIDBVR"
+		(property "Value" "TLV9061IDBVR"
 			(at 295.91 187.96 0)
 			(show_name no)
@@
 			)
 		)
-		(property "Manufacturer Part Number" "TLV9061SIDBVR"
+		(property "Manufacturer Part Number" "TLV9061IDBVR"
 			(at 289.56 193.04 0)
 			(hide yes)
@@
 			)
 		)
-		(property "Supplier Part Number" "296-53200-1-ND"
+		(property "Supplier Part Number" "296-52284-1-ND"
 			(at 289.56 193.04 0)
 			(hide yes)
