File: powerSupplies.kicad_sch (KiCad schematic)
At the start: 64 parts, among them U301 LMR54410DBVR, U302 LMR54410DBVR, U303 SPX3819M5-L-3-3/TR, U304 SPX3819M5-L-3-3/TR, U305 LDLN025M33R, U306 LM66100DCK

Commit message: Update sch v1.0
Parts:
- TP306: footprint 0_testpoints:TestPoint_NoSlik_D1.0mm_Top -> 0_testpoints:TestPoint_NoSlik_D1.0mm_Bottom
Changed lines of the file:
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@@
 			)
 		)
-		(property "Footprint" "0_testpoints:TestPoint_NoSlik_D1.0mm_Top"
+		(property "Footprint" "0_testpoints:TestPoint_NoSlik_D1.0mm_Bottom"
 			(at 80.01 242.57 0)
 			(hide yes)

Commit message: Modified part number
Added 2nd Supplier
Added 2nd Mfr, Mfr NO.
Parts:
- LD301: Manufacturer LITE-ON -> (none); Manufacturer 2nd (none) -> LITE-ON; Manufacturer Part Number LTST-C191TGKT -> (none); Manufacturer Part Number 2nd (none) -> LTST-C191TGKT; Supplier ES -> (none); Supplier 2nd (none) -> Electronisc Source; Supplier Part Number 0013-0123-1 -> (none); Supplier Part Number 2nd (none) -> 0013-0123-1; now in the parts list
- R303: Manufacturer 2nd (none) -> ROYALOHM; Manufacturer Part Number 2nd (none) -> 0402WGF1623TCE; Supplier 2nd (none) -> Electronisc Source; Supplier Part Number 2nd (none) -> 0150-4690-4
- R312: Manufacturer 2nd (none) -> ROYALOHM; Manufacturer Part Number 2nd (none) -> 0402WGF5111TCE; Supplier 2nd (none) -> Electronisc Source; Supplier Part Number 2nd (none) -> 0150-3609-4
