File: powerSupplies.kicad_sch (KiCad schematic)
At the start: 64 parts, among them U301 LMR54410DBVR, U302 LMR54410DBVR, U303 SPX3819M5-L-3-3/TR, U304 SPX3819M5-L-3-3/TR, U305 LDLN025M33R, U306 LM66100DCK

Commit message: Updated Schematic v1.0
Parts:
- D301: now left out of the parts list
Changed lines of the file:
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@@
 		(in_bom no)
 		(on_board yes)
-		(in_pos_files yes)
+		(in_pos_files no)
 		(dnp no)
 		(property "Reference" "NT305"
@@
 		(in_bom no)
 		(on_board yes)
-		(in_pos_files yes)
+		(in_pos_files no)
 		(dnp no)
 		(property "Reference" "NT303"
@@
 		(body_style 1)
 		(exclude_from_sim no)
-		(in_bom yes)
+		(in_bom no)
 		(on_board yes)
 		(in_pos_files yes)
@@
 		(in_bom no)
 		(on_board yes)
-		(in_pos_files yes)
+		(in_pos_files no)
 		(dnp no)
 		(property "Reference" "NT304"
