File: powerSupplies.kicad_sch (KiCad schematic)
At the start: 64 parts, among them U301 LMR54410DBVR, U302 LMR54410DBVR, U303 SPX3819M5-L-3-3/TR, U304 SPX3819M5-L-3-3/TR, U305 LDLN025M33R, U306 LM66100DCK

Commit message: Migrate Symbol Librarys
Parts:
- D301: symbol 0_diode:BAT60JFILM -> 0_Diode:BAT60JFILM
- U301, U302: symbol 0_buck:LMR54410DBV -> 0_Buck:LMR54410DBV
- U303, U304: symbol 0_regulators:SPX3819M5-L-3-3 -> 0_Regulators:SPX3819M5-L-3-3
- U305: symbol 0_regulators:LDLN025M33R -> 0_Regulators:LDLN025M33R
Changed lines of the file:
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@@
 	)
 	(symbol
-		(lib_id "0_regulators:LDLN025M33R")
+		(lib_id "0_Regulators:LDLN025M33R")
 		(at 340.36 163.83 0)
 		(unit 1)
@@
 	)
 	(symbol
-		(lib_id "0_buck:LMR54410DBV")
+		(lib_id "0_Buck:LMR54410DBV")
 		(at 147.32 50.8 0)
 		(unit 1)
@@
 	)
 	(symbol
-		(lib_id "0_diode:BAT60JFILM")
+		(lib_id "0_Diode:BAT60JFILM")
 		(at 186.69 203.2 180)
 		(unit 1)
@@
 	)
 	(symbol
-		(lib_id "0_buck:LMR54410DBV")
+		(lib_id "0_Buck:LMR54410DBV")
 		(at 147.32 129.54 0)
 		(unit 1)
@@
 	)
 	(symbol
-		(lib_id "0_regulators:SPX3819M5-L-3-3")
+		(lib_id "0_Regulators:SPX3819M5-L-3-3")
 		(at 328.93 113.03 0)
 		(unit 1)
@@
 	)
 	(symbol
-		(lib_id "0_regulators:SPX3819M5-L-3-3")
+		(lib_id "0_Regulators:SPX3819M5-L-3-3")
 		(at 330.2 59.69 0)
 		(unit 1)
