File: power_connectors.kicad_sch (KiCad schematic)
At the start: 10 parts, among them CN201 04A2, CN202 04A2, CN203 04A2, CN204 04A2, CN205 SMA-J-P-H-ST-EM1

Commit message: Modified part number
Added 2nd Supplier
Added 2nd Mfr, Mfr NO.
Parts:
- R202: Manufacturer 2nd (none) -> ROYALOHM; Manufacturer Part Number 2nd (none) -> 0402WGF499JTCE; Supplier 2nd (none) -> Electronisc Source; Supplier Part Number 2nd (none) -> 0150-4765-9
