File: power_connectors.kicad_sch (KiCad schematic)
At the start: 10 parts, among them CN201 04A2, CN202 04A2, CN203 04A2, CN204 04A2, CN205 SMA-J-P-H-ST-EM1

Commit message: Update power_connectors.kicad_sch
Other:
- note removed: "30V 12A MAX"
Changed lines of the file:
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@@
 		)
 	)
-	(text "30V 12A MAX "
+	(text "30V 20A MAX "
 		(exclude_from_sim no)
 		(at 163.83 104.14 0)

Commit message: Migrate Symbol Librarys
Parts:
- CN201, CN202, CN203, CN204: symbol 0_connectors:Conn_02x02_Top_Bottom -> 0_Connectors:Conn_02x02_Top_Bottom
- D201, D202: symbol 0_protection:SMBJ30A -> 0_Protection:SMBJ30A
Changed lines of the file:
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@@
 	)
 	(symbol
-		(lib_id "0_connectors:Conn_02x02_Top_Bottom")
+		(lib_id "0_Connectors:Conn_02x02_Top_Bottom")
 		(at 303.53 114.3 90)
 		(unit 1)
@@
 	)
 	(symbol
-		(lib_id "0_connectors:Conn_02x02_Top_Bottom")
+		(lib_id "0_Connectors:Conn_02x02_Top_Bottom")
 		(at 99.06 114.3 90)
 		(unit 1)
@@
 	)
 	(symbol
-		(lib_id "0_connectors:Conn_02x02_Top_Bottom")
+		(lib_id "0_Connectors:Conn_02x02_Top_Bottom")
 		(at 111.76 114.3 90)
 		(unit 1)
@@
 	)
 	(symbol
-		(lib_id "0_protection:SMBJ30A")
+		(lib_id "0_Protection:SMBJ30A")
 		(at 287.02 115.57 270)
 		(unit 1)
@@
 	)
 	(symbol
-		(lib_id "0_protection:SMBJ30A")
+		(lib_id "0_Protection:SMBJ30A")
 		(at 128.27 115.57 270)
 		(unit 1)
@@
 	)
 	(symbol
-		(lib_id "0_connectors:Conn_02x02_Top_Bottom")
+		(lib_id "0_Connectors:Conn_02x02_Top_Bottom")
 		(at 316.23 114.3 90)
 		(unit 1)
