File: power_state.kicad_sch (KiCad schematic)
At the start: 103 parts, among them Q101 BSZ018N04LS6, Q102 IQE013N04LM6, Q103 BSZ018N04LS6, Q104 IQE013N04LM6, Q105 GS2N7002KW, Q106 GS2N7002KW, U101 UCC27282DRC, U102 ACS37030LLZATR-040B3, U103 UCC27282DRC, U104 ACS37030LLZATR-040B3, U106 INA187A1IDBVR

Commit message: Update sch v1.0
Other:
- note removed: "Place start winding dot mark to sw node side"
Changed lines of the file:
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@@
-		)
-	)
-	(text "Place start winding dot mark to sw node side"
-		(exclude_from_sim no)
-		(at 227.965 108.585 0)
-		(effects
-			(font
-				(size 1.27 1.27)
-				(color 0 0 194 1)
-			)
 		)
 	)
@@
 	(text_box "LAYOUT NOTE:\n\nMake the Size of SW Node small as possible but sufficient to handle current"
 		(exclude_from_sim no)
-		(at 241.3 92.71 0)
+		(at 181.61 88.9 0)
 		(size 25.4 12.7)
 		(margins 0.9525 0.9525 0.9525 0.9525)
@@
 			)
 			(justify left top)
-		)
-	)
-	(text_box "LAYOUT NOTE:\n\nPlace the bootstap capacitor as close to HB, HS pin as possible."
-		(exclude_from_sim no)
-		(at 212.09 92.71 0)
-		(size 24.13 12.7)
-		(margins 0.9525 0.9525 0.9525 0.9525)
-		(stroke
-			(width 0.5)
-			(type solid)
-			(color 0 0 194 1)
-		)
-		(fill
-			(type color)
-			(color 255 255 194 1)
-		)
-		(effects
-			(font
-				(face "Century Gothic")
-				(size 1.27 1.27)
-				(thickness 0.1588)
-				(bold yes)
-				(color 0 0 194 1)
-			)
-			(justify left top)

Commit message: Modified part number
Added 2nd Supplier
Added 2nd Mfr, Mfr NO.
Parts:
- C116, C128: Manufacturer 2nd (none) -> Murata; Manufacturer Part Number 2nd (none) -> GCM1555C1H101FA16D; Supplier 2nd (none) -> Electronisc Source; Supplier Part Number 2nd (none) -> 0160-1291-2
- R105, R111: Manufacturer 2nd (none) -> ROYALOHM; Manufacturer Part Number 2nd (none) -> CQ02WGF1000TCE; Supplier 2nd (none) -> Electronisc Source; Supplier Part Number 2nd (none) -> 0150-4399-1
- R106, R112: Manufacturer 2nd (none) -> ROYALOHM; Manufacturer Part Number 2nd (none) -> CQ02WGF1003TCE; Supplier 2nd (none) -> Electronisc Source; Supplier Part Number 2nd (none) -> 0150-4421-7
- R107, R108, R113, R114: Manufacturer ROYALOHM -> (none); Manufacturer 2nd (none) -> ROYALOHM; Manufacturer Part Number 0603WAF221KT5E -> (none); Manufacturer Part Number 2nd (none) -> 0603WAF221KT5E; Supplier ES -> (none); Supplier 2nd (none) -> Electronisc Source; Supplier Part Number 0150-4758-2 -> (none); Supplier Part Number 2nd (none) -> 0150-4758-2; now in the parts list
- R116, R118: Manufacturer 2nd (none) -> YAGEO; Manufacturer Part Number 2nd (none) -> RC0603FR-079K09L; Supplier 2nd (none) -> Electronisc Source; Supplier Part Number 2nd (none) -> 0151-0863-5
