File: power_state.kicad_sch (KiCad schematic)
At the start: 101 parts, among them Q101 BSZ018N04LS6, Q102 IQE013N04LM6, Q103 BSZ018N04LS6, Q104 IQE013N04LM6, U101 UCC27282DRC, U102 ACS37030LLZATR-040B3, U103 UCC27282DRC, U104 ACS37030LLZATR-040B3, U106 INA187A1IDBVR

Commit message: Update revision
- Shc.
- Render images
Parts:
- R104, R110: now left out of the parts list
Other:
- note added: "A1's GAIN: 20V/V I = 1/20 x Vout/0.005"
- note removed: "A1 GAIN: 20V/V"
Changed lines of the file:
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@@
 	(text "ESD Sensitive"
 		(exclude_from_sim no)
-		(at 247.65 274.32 0)
+		(at 223.52 316.23 0)
 		(effects
 			(font
@@
 	(text "Hot surface"
 		(exclude_from_sim no)
-		(at 233.68 274.32 0)
+		(at 209.55 316.23 0)
 		(effects
 			(font
@@
 		)
 	)
-	(text "A1 GAIN: 20V/V"
+	(text "A1's GAIN: 20V/V\nI = 1/20 x Vout/0.005"
 		(exclude_from_sim no)
-		(at 95.25 74.93 0)
+		(at 88.9 74.93 0)
 		(effects
 			(font
@@
 				(thickness 0.1588)
 			)
+			(justify left)
 		)
 	)
@@
 	(symbol
 		(lib_id "Graphic:SYM_Hot_Large")
-		(at 233.68 266.7 0)
+		(at 209.55 308.61 0)
 		(unit 1)
 		(body_style 1)
@@
 		(fields_autoplaced yes)
 		(property "Reference" "G101"
-			(at 233.68 261.62 0)
+			(at 209.55 303.53 0)
 			(hide yes)
 			(show_name no)
@@
 		)
 		(property "Value" "SYM_Hot_Large"
-			(at 233.68 273.05 0)
+			(at 209.55 314.96 0)
 			(hide yes)
 			(show_name no)
@@
 		)
 		(property "Footprint" "0_symbols:hot_surface"
-			(at 233.68 271.78 0)
+			(at 209.55 313.69 0)
 			(hide yes)
 			(show_name no)
@@
 		)
 		(property "Datasheet" ""
-			(at 234.442 271.78 0)
+			(at 210.312 313.69 0)
 			(hide yes)
 			(show_name no)
@@
 		)
 		(property "Description" "Hot surface warning symbol, large"
-			(at 233.68 266.7 0)
+			(at 209.55 308.61 0)
 			(hide yes)
 			(show_name no)
@@
 		(body_style 1)
 		(exclude_from_sim no)
-		(in_bom yes)
+		(in_bom no)
 		(on_board yes)
 		(in_pos_files yes)
@@
 		(body_style 1)
 		(exclude_from_sim no)
-		(in_bom yes)
+		(in_bom no)
 		(on_board yes)
 		(in_pos_files yes)
@@
 	(symbol
 		(lib_id "Graphic:SYM_ESD_Large")
-		(at 247.65 266.7 0)
+		(at 223.52 308.61 0)
 		(unit 1)
 		(body_style 1)
@@
 		(fields_autoplaced yes)
 		(property "Reference" "G102"
-			(at 247.65 261.62 0)
+			(at 223.52 303.53 0)
 			(hide yes)
 			(show_name no)
@@
 		)
 		(property "Value" "SYM_ESD_Large"
-			(at 247.65 273.05 0)
+			(at 223.52 314.96 0)
 			(hide yes)
 			(show_name no)
@@
 		)
 		(property "Footprint" "Symbol:ESD-Logo_6.6x6mm_SilkScreen"
-			(at 247.523 267.462 0)
+			(at 223.393 309.372 0)
 			(hide yes)
 			(show_name no)
@@
 		)
 		(property "Datasheet" ""
-			(at 247.523 267.462 0)
+			(at 223.393 309.372 0)
 			(hide yes)
 			(show_name no)
@@
 		)
 		(property "Description" "ESD warning/\"Do not touch\" symbol, large"
-			(at 247.65 266.7 0)
+			(at 223.52 308.61 0)
 			(hide yes)
 			(show_name no)

Commit message: Migrate Symbol Librarys
Parts:
- D101, D102, D103, D104: symbol 0_diode:BAT54XV2T5G -> 0_Diode:BAT54XV2T5G
- G103: symbol 0_miscellaneous:BlankSymbol -> 0_Miscellaneous:BlankSymbol
- Q101, Q103: symbol 0_infineon_MOSFET:BSZ018N04LS6 -> 0_Infineon_MOSFET:BSZ018N04LS6
- Q102, Q104: symbol 0_infineon_MOSFET:IQE013N04LM6 -> 0_Infineon_MOSFET:IQE013N04LM6
- U101, U103: symbol 0_gateDrivers:UCC27282DRCR -> 0_GateDrivers:UCC27282DRCR
- U102, U104: symbol 0_currentSensors:ACS37030LLZATR -> 0_CurrentSensors:ACS37030LLZATR
- U106: symbol 0_currentSensors:INA187Ax -> 0_CurrentSensors:INA187Ax
Changed lines of the file:
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@@
 	)
 	(symbol
-		(lib_id "0_diode:BAT54XV2T5G")
+		(lib_id "0_Diode:BAT54XV2T5G")
 		(at 138.43 143.51 0)
 		(unit 1)
@@
 	)
 	(symbol
-		(lib_id "0_currentSensors:ACS37030LLZATR")
+		(lib_id "0_CurrentSensors:ACS37030LLZATR")
 		(at 247.65 201.93 0)
 		(unit 1)
@@
 	)
 	(symbol
-		(lib_id "0_currentSensors:ACS37030LLZATR")
+		(lib_id "0_CurrentSensors:ACS37030LLZATR")
 		(at 247.65 129.54 0)
 		(unit 1)
@@
 	)
 	(symbol
-		(lib_id "0_diode:BAT54XV2T5G")
+		(lib_id "0_Diode:BAT54XV2T5G")
 		(at 138.43 118.11 0)
 		(unit 1)
@@
 	)
 	(symbol
-		(lib_id "0_infineon_MOSFET:IQE013N04LM6")
+		(lib_id "0_Infineon_MOSFET:IQE013N04LM6")
 		(at 162.56 222.25 0)
 		(unit 1)
@@
 	)
 	(symbol
-		(lib_id "0_currentSensors:INA187Ax")
+		(lib_id "0_CurrentSensors:INA187Ax")
 		(at 81.28 55.88 0)
 		(unit 1)
@@
 			)
 		)
+		(property "Manufacturer 2nd" ""
+			(at 81.28 55.88 0)
+			(hide yes)
+			(show_name no)
+			(do_not_autoplace no)
+			(effects
+				(font
+					(size 1.27 1.27)
+				)
+			)
+		)
+		(property "Manufacturer Part Number 2nd" ""
+			(at 81.28 55.88 0)
+			(hide yes)
+			(show_name no)
+			(do_not_autoplace no)
+			(effects
+				(font
+					(size 1.27 1.27)
+				)
+			)
+		)
+		(property "Supplier Part Number 2nd" ""
+			(at 81.28 55.88 0)
+			(hide yes)
+			(show_name no)
+			(do_not_autoplace no)
+			(effects
+				(font
+					(size 1.27 1.27)
+				)
+			)
+		)
+		(property "Supplier 2nd" ""
+			(at 81.28 55.88 0)
+			(hide yes)
+			(show_name no)
+			(do_not_autoplace no)
+			(effects
+				(font
+					(size 1.27 1.27)
+				)
+			)
+		)
 		(pin "6"
 		)
@@
 	)
 	(symbol
-		(lib_id "0_infineon_MOSFET:IQE013N04LM6")
+		(lib_id "0_Infineon_MOSFET:IQE013N04LM6")
 		(at 162.56 149.86 0)
 		(unit 1)
@@
 	)
 	(symbol
-		(lib_id "0_infineon_MOSFET:BSZ018N04LS6")
+		(lib_id "0_Infineon_MOSFET:BSZ018N04LS6")
 		(at 162.56 196.85 0)
 		(unit 1)
@@
 	)
 	(symbol
-		(lib_id "0_diode:BAT54XV2T5G")
+		(lib_id "0_Diode:BAT54XV2T5G")
 		(at 138.43 215.9 0)
 		(unit 1)
@@
 	)
 	(symbol
-		(lib_id "0_infineon_MOSFET:BSZ018N04LS6")
+		(lib_id "0_Infineon_MOSFET:BSZ018N04LS6")
 		(at 162.56 124.46 0)
 		(unit 1)
@@
 	)
 	(symbol
-		(lib_id "0_miscellaneous:BlankSymbol")
+		(lib_id "0_Miscellaneous:BlankSymbol")
 		(at 241.3 308.61 0)
 		(unit 1)
@@
 	)
 	(symbol
-		(lib_id "0_gateDrivers:UCC27282DRCR")
+		(lib_id "0_GateDrivers:UCC27282DRCR")
 		(at 97.79 190.5 0)
 		(unit 1)
@@
 	)
 	(symbol
-		(lib_id "0_gateDrivers:UCC27282DRCR")
+		(lib_id "0_GateDrivers:UCC27282DRCR")
 		(at 97.79 118.11 0)
 		(unit 1)
@@
 	)
 	(symbol
-		(lib_id "0_diode:BAT54XV2T5G")
+		(lib_id "0_Diode:BAT54XV2T5G")
 		(at 138.43 190.5 0)
 		(unit 1)
