File: user_LED.kicad_sch (KiCad schematic)
At the start: 22 parts, among them Q801 GS2N7002KW, Q802 GS2N7002KW, Q803 GS2N7002KW, Q804 GS2N7002KW

Commit message: Modified part number
Added 2nd Supplier
Added 2nd Mfr, Mfr NO.
Parts:
- LD801, LD804: Manufacturer LITE-ON -> (none); Manufacturer 2nd (none) -> LITE-ON; Manufacturer Part Number LTST-C190KFKT -> (none); Manufacturer Part Number 2nd (none) -> LTST-C190KFKT; Supplier ES -> (none); Supplier 2nd (none) -> Electronisc Source; Supplier Part Number 0013-0112-6 -> (none); Supplier Part Number 2nd (none) -> 0013-0112-6; now in the parts list
- LD802: Manufacturer LITE-ON -> (none); Manufacturer 2nd (none) -> LITE-ON; Manufacturer Part Number LTST-C191TGKT -> (none); Manufacturer Part Number 2nd (none) -> LTST-C191TGKT; Supplier ES -> (none); Supplier 2nd (none) -> Electronisc Source; Supplier Part Number 0013-0123-1 -> (none); Supplier Part Number 2nd (none) -> 0013-0123-1; now in the parts list
- LD803: Manufacturer LITE-ON -> (none); Manufacturer 2nd (none) -> LITE-ON; Manufacturer Part Number LTST-C191KRKT -> (none); Manufacturer Part Number 2nd (none) -> LTST-C191KRKT; Supplier ES -> (none); Supplier 2nd (none) -> Electronisc Source; Supplier Part Number 0013-0100-4 -> (none); Supplier Part Number 2nd (none) -> 0013-0100-4; now in the parts list
- R802, R803: Manufacturer 2nd (none) -> ROYALOHM; Manufacturer Part Number 2nd (none) -> 0402WGF1001TCE; Supplier 2nd (none) -> Electronisc Source; Supplier Part Number 2nd (none) -> 0150-3602-3
- R805, R806, R807, R808: Manufacturer 2nd (none) -> ROYALOHM; Manufacturer Part Number 2nd (none) -> CQ02WGF1000TCE; Supplier 2nd (none) -> Electronisc Source; Supplier Part Number 2nd (none) -> 0150-4399-1
- R809, R810, R811, R812: Manufacturer 2nd (none) -> ROYALOHM; Manufacturer Part Number 2nd (none) -> CQ02WGF1003TCE; Supplier 2nd (none) -> Electronisc Source; Supplier Part Number 2nd (none) -> 0150-4421-7
