File: user_LED.kicad_sch (KiCad schematic)
At the start: 22 parts, among them Q801 GS2N7002KW, Q802 GS2N7002KW, Q803 GS2N7002KW, Q804 GS2N7002KW

Commit message: Migrate Symbol Librarys
Parts:
- Q801, Q802, Q803, Q804: symbol 0_mosfet:GS2N7002KW -> 0_Mosfet:GS2N7002KW
Changed lines of the file:
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@@
 	)
 	(symbol
-		(lib_id "0_mosfet:GS2N7002KW")
+		(lib_id "0_Mosfet:GS2N7002KW")
 		(at 157.48 113.03 0)
 		(unit 1)
@@
 	)
 	(symbol
-		(lib_id "0_mosfet:GS2N7002KW")
+		(lib_id "0_Mosfet:GS2N7002KW")
 		(at 213.36 214.63 0)
 		(unit 1)
@@
 	)
 	(symbol
-		(lib_id "0_mosfet:GS2N7002KW")
+		(lib_id "0_Mosfet:GS2N7002KW")
 		(at 213.36 113.03 0)
 		(unit 1)
@@
 	)
 	(symbol
-		(lib_id "0_mosfet:GS2N7002KW")
+		(lib_id "0_Mosfet:GS2N7002KW")
 		(at 271.78 113.03 0)
 		(unit 1)
