File: 2Phase_SynchBuck.kicad_pcb (KiCad board)
At the start: 4 copper layers, 100 x 67 mm, 306 parts, among them CN201 04A2, CN202 04A2, CN203 04A2, CN204 04A2, CN205 SMA-J-P-H-ST-EM1, CN701 USB4215-03-A, CN702 Conn_JTAG_STDC10, CN703 FFC2B28-16-G, CN704 FFC2B28-04-G, Q101 BSZ018N04LS6, Q102 IQE013N04LM6, Q103 BSZ018N04LS6, Q104 IQE013N04LM6, Q801 GS2N7002KW, Q802 GS2N7002KW, Q803 GS2N7002KW, Q804 GS2N7002KW, SW901 SW_SPDT, U101 UCC27282DRC, U102 ACS37030LLZATR-040B3, U103 UCC27282DRC, U104 ACS37030LLZATR-040B3, U106 INA187A1IDBVR, U301 LMR54410DBVR, U302 LMR54410DBVR, U303 SPX3819M5-L-3-3/TR, U304 SPX3819M5-L-3-3/TR, U305 LDLN025M33R, U306 LM66100DCK, U401 STM32G474RET6, U402 MCP1501T-30E, U601 TLV9061SIDBVR, U602 TLV9061SIDBVR, U701 USBLC6-2SC6, X501 ABM11W-24MHz-8

Commit message: Update 2Phase_SynchBuck.kicad_pcb
Change TP? Description
Other:
- board text added: "GND GND +9V +5V +3V3 GND Analog Vout GND PC11 PC12 PD2 PB3 PB4 PB5 TX RX DAC1 DAC2"
- board text added: "Gate HS 1 Gate LS 1 Gate HS 2 Gate LS 2 Vin Filter Switch-node 1 Switch-node 2 VREF1 VREF2 IL1 IL2 I_IN +USB +A3V3 +S3V3 HTIM_E1 Analog VIN GND"
- board text added: "L1 (Signal) (Scale 1:1)"
- board text added: "L2 (GND) (Scale 1:1)"
- board text added: "L3 (GND) (Scale 1:1)"
- board text added: "L4 (Signal) (Scale 1:1)"
- board text added: "TP101 TP102 TP103 TP104 TP105 TP106 TP107 TP108 TP109 TP110 TP111 TP112 TP303 TP305 TP306 TP501 TP602 TP604"
- board text added: "TP113 TP114 TP301 TP302 TP304 TP307 TP601 TP603 TP701 TP702 TP703 TP704 TP705 TP706 TP707 TP708 TP709 TP710"
- board text removed: "+9V +5V +3V3 Analog Vout GND PC11 PC12 PD2 PB3 PB4 PB5 TX RX DAC1 DAC2"
- board text removed: "Gate HS 1 Gate LS 1 Gate HS 2 Gate LS 2 Vin Filter Switch-node 1 Switch-node 2 VREF1 VREF2 IL1 IL2 I_IN GND GND +USB +A3V3 +S3V3 GND HTIM_E1 Analog VIN GND"
- board text removed: "L1 (Signal) (Scale 2:1)"
- board text removed: "L2 (GND) (Scale 2:1)"
- board text removed: "L3 (GND) (Scale 2:1)"
- board text removed: "L4 (Signal) (Scale 2:1)"
- board text removed: "TP101 TP102 TP103 TP104 TP105 TP106 TP107 TP108 TP109 TP110 TP111 TP112 TP113 TP114 TP303 TP305 TP306 TP307 TP501 TP602 TP604"
- board text removed: "TP301 TP302 TP304 TP601 TP603 TP701 TP702 TP703 TP704 TP705 TP706 TP707 TP708 TP709 TP710"
