File: Block_diagram.kicad_sch (KiCad schematic)
At the start: 0 parts

Commit message: Update sch v1.0
Other:
- note added: "28V"
- note removed: "30V"
Changed lines of the file:
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@@
 		)
 	)
-	(text "30V"
+	(text "28V"
 		(exclude_from_sim no)
 		(at 113.03 162.56 0)
@@
 		)
 	)
-	(text "30V"
+	(text "28V"
 		(exclude_from_sim no)
 		(at 100.33 137.16 0)
@@
 		)
 	)
-	(text_box "PC9, PB15"
+	(text_box "PA10, PC9"
 		(exclude_from_sim no)
 		(at 246.38 115.57 0)
