File: RevHistory.kicad_sch (KiCad schematic)
At the start: 0 parts

Commit message: Update revision
- Shc.
- Render images
Other:
- note added: "(28/06/2026) - Remove the Mosfet that Enable the ICs Gate Driver (p.1) - Change ADC input Capacitor 47pF to 1nF. (p.6) - Change op-amp U601 U602 to correctly part number (p.6)"
- note removed: "(28/06/2026) - Removed the Mosfet that Enable the ICs Gate Driver (p.1) - Changed ADC input Capacitor 47pF to 1nF. (p.6)"
Changed lines of the file:
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@@
 		(comment 1 "Revision History")
 	)
-	(text "(28/06/2026) \n- Removed the Mosfet that Enable the ICs Gate Driver (p.1)\n- Changed ADC input Capacitor 47pF to 1nF. (p.6)"
+	(text "(28/06/2026) \n- Remove the Mosfet that Enable the ICs Gate Driver (p.1)\n- Change ADC input Capacitor 47pF to 1nF. (p.6)\n- Change op-amp U601 U602 to correctly part number (p.6)"
 		(exclude_from_sim no)
-		(at 41.91 83.82 0)
+		(at 41.91 85.09 0)
 		(effects
 			(font

Commit message: Update RevHistory.kicad_sch
Other:
- note added: "(28/06/2026) - Remove the MOSFETs that Enable the ICs Gate Driver and connect directly. (p.1) - Change ADC input Capacitor 47pF to 1nF. (p.6) - Change OP-AMP U601 U602 to correctly part number (p.6)"
- note removed: "(28/06/2026) - Remove the Mosfet that Enable the ICs Gate Driver (p.1) - Change ADC input Capacitor 47pF to 1nF. (p.6) - Change op-amp U601 U602 to correctly part number (p.6)"
Changed lines of the file:
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@@
 		(comment 1 "Revision History")
 	)
-	(text "(28/06/2026) \n- Remove the Mosfet that Enable the ICs Gate Driver (p.1)\n- Change ADC input Capacitor 47pF to 1nF. (p.6)\n- Change op-amp U601 U602 to correctly part number (p.6)"
+	(text "(28/06/2026) \n- Remove the MOSFETs that Enable the ICs Gate Driver and connect directly. (p.1)\n- Change ADC input Capacitor 47pF to 1nF. (p.6)\n- Change OP-AMP U601 U602 to correctly part number (p.6)"
 		(exclude_from_sim no)
 		(at 41.91 85.09 0)
