File: pwr_sequencing.kicad_sch (KiCad schematic)
At the start: 0 parts

Commit message: Migrate Symbol Librarys
Other:
- note added: "(1) Enable 5V Buck"
- note added: "(2) Enable 9V Buck"
- note added: "4.5V"
- note added: "Not measured"
- note removed: "1.2V"
- note removed: "> NORMAL OPERATING POINT"
