File: user_interface.kicad_sch (KiCad schematic)
At the start: 14 parts, among them SW901 SW_SPDT

Commit message: Migrate Symbol Librarys
Parts:
- D901, D902, D903: symbol 0_protection:ESD5Z3V3 -> 0_Protection:ESD5Z3V3
Changed lines of the file:
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@@
 	)
 	(symbol
-		(lib_id "0_protection:ESD5Z3V3")
+		(lib_id "0_Protection:ESD5Z3V3")
 		(at 260.35 107.95 270)
 		(unit 1)
@@
 	)
 	(symbol
-		(lib_id "0_protection:ESD5Z3V3")
+		(lib_id "0_Protection:ESD5Z3V3")
 		(at 156.21 194.31 270)
 		(unit 1)
@@
 	)
 	(symbol
-		(lib_id "0_protection:ESD5Z3V3")
+		(lib_id "0_Protection:ESD5Z3V3")
 		(at 147.32 113.03 270)
 		(unit 1)
